Commit message: created initial urdf file for inverted pendulum bot need to add collision and gazebo integration

File: urdf/inverted_pendulum.urdf (robot description, URDF)
Before this commit: robot myfirst, 1 links, 0 joints
Links:
- added link left_wheel_link; visual cylinder length=0.2 radius=0.2
- added link right_wheel_link; visual cylinder length=0.2 radius=0.2
Joints:
- added joint left_wheel_joint: type continuous, parent base_link, child left_wheel_link, origin xyz=0.2 0 -0.3 rpy=0 1.6 0, axis 0 0 1
- added joint right_wheel_joint: type continuous, parent base_link, child right_wheel_link, origin xyz=-0.2 0 -0.3 rpy=0 -1.6 0, axis 0 0 1
